File: _autosave-MLGC210815.sch (KiCad schematic (older format))
At the start: 53 parts, among them J1 PinStrip_01x06_Male, U1 PIC32MX170F256B-ISS

Commit message: update
Parts:
- removed C? (x2): C0805_1uF_X7R, Passive:C0805, symbol MLGC210815-rescue:C0805_1uF_X7R-Passive
- added C? (x2): Capacitator_0603_2.2uF_X5R, Passive:C0603, symbol Passive:Capacitator_0603_2.2uF_X5R
- added D?: LED0805_KP-2012SGC, Passive:R0805, symbol MLGC210815-rescue:LED0805_KP-2012SGC-Passive
Connections:
- net labels added: AN1, INT1, SCL1, SDA1, U1TX
- net labels removed: SCL, SDA
- wire segments 158 -> 144
- no-connect marks 0 -> 6
Other:
- note removed: "LIS2DE12"
- note removed: "SI2315BDS-T1-E3"
- moved on the sheet: C2, C?, R?, Y?
