File: _autosave-MLGC210815.sch (KiCad schematic (older format))
At the start: 108 parts, among them J1 PinStrip_01x06_Male, J2 USB-B-04PFHTW, Q1 P-MOSFET_SI2315BDS-T1-E3, Q2 NPN_BC817, Q3 NPN_BC817, Q4 P-MOSFET_SI2315BDS-T1-E3, SW1 Switch-Tact_OMRON-B3F-3100, SW2 Switch-Tact_OMRON-B3F-3100, SW3 Switch-Tact_OMRON-B3F-3100, U1 PIC32MX170F256B-ISS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

Commit message: updATE
Parts:
- U3: footprint Package_TO_SOT_SMD:SOT-23 -> Semiconductor:SOT-23; symbol MLGC210815-rescue:LDO-MCP1700T-3302E_TT-Others -> Others:LDO_MCP1700T-3302E_TT
Changed lines of the file:
@@
 $EndComp
 $Comp
-L MLGC210815-rescue:LDO-MCP1700T-3302E_TT-Others U3
+L Others:LDO_MCP1700T-3302E_TT U3
 U 1 1 612BD3E2
 P 2150 7100
 F 0 "U3" H 2300 7250 50  0000 C CNN
 F 1 "LDO-MCP1700T-3302E_TT-Others" H 2150 7225 50  0001 L CNN
-F 2 "Package_TO_SOT_SMD:SOT-23" H 2150 7325 50  0001 C CNN
+F 2 "Semiconductor:SOT-23" H 2150 7325 50  0001 C CNN
 F 3 "D:\\@@@!ProjectS\\Cirucits\\KiCad\\Datasheet\\MICROCHIP MCP1700T3302ETT.pdf" H 2150 7100 50  0001 C CNN
 F 4 "MCP1700T-3302E/TT" H 2150 6650 50  0000 C CNN "Comment"

Commit message: update
Parts:
- removed C14: Capacitator_0603_47nF_X7R, Passive:C_0603, symbol Passive:Capacitator_0603_47nF_X7R
- removed R16: Resistor_0603_4K70, Passive:R_0603, symbol Passive:Resistor_0603_4K70
- removed R17: Resistor_0603_9K10, Passive:R_0603, symbol Passive:Resistor_0603_9K10
- removed R18: Resistor_0603_10R0, Passive:R_0603, symbol Passive:Resistor_0603_10R0
- removed R44: Resistor_0603_0R00, Passive:R_0603, symbol Passive:Resistor_0603_0R00
- removed Y1: Crystal_HC49SM_8MHz, Passive:Crystal_SMD_HC49-SD, symbol Passive:Crystal_HC49SM_8MHz
- added J3, J4: PinHeader_01x01_Male, Connectors:PinHeader_1x01_P2.54mm_Horizontal, symbol Connectors:PinHeader_01x01_Male
- added J5: PinHeader_01x02_Male, Connectors:PinHeader_1x02_P2.54mm_Vertical, symbol Connectors:PinHeader_01x02_Male
- added L3: Filter_0603_CB03YTYH101, Passive:L_0603, symbol Passive:Filter_0603_CB03YTYH101
- added R16: Resistor_0603_0R00, Passive:R_0603, symbol Passive:Resistor_0603_0R00
- added R44: Resistor_0603_220R, Passive:R_0603, symbol Passive:Resistor_0603_220R
- added R45: Resistor_0603_1K00, Passive:R_0603, symbol Passive:Resistor_0603_1K00
- added Y1: Crystal_SMD3225_12MHz, Passive:Crystal_SMD_3225, symbol Passive:Crystal_SMD3225_12MHz
- B1: value BATTERY_CELLEVIA-L402036-Others -> BATTERY_L402036; symbol MLGC210815-rescue:BATTERY_CELLEVIA-L402036-Others -> Others:BATTERY_L402036
- C1, C10, C11, C2, C6, C8: value Capacitator_0805_100nF_X7R -> Capacitator_0603_100nF_X7R; footprint Passive:C_0805 -> Passive:C_0603; symbol Passive:Capacitator_0805_100nF_X7R -> Passive:Capacitator_0603_100nF_X7R; ManufacturerPartNo CC0805KRX7R9BB104 -> CC0603KRX7R9BB104; Supplier FAR-3019949;LOM-82-01-25 -> LOM-82-03-47;TME-CC0603KRX7R9BB104;
- C12, C16, C26, C34, C35, C36, C9: value Capacitator_0805_1uF_X7R -> Capacitator_0603_1uF_X7R; symbol Passive:Capacitator_0805_1uF_X7R -> Passive:Capacitator_0603_1uF_X7R; ManufacturerPartNo CC0603KRX7R7BB105 -> CC0603KRX7R7BB105;
- C20, C21, C22: Comment 100nF -> 10nF
- C3: value Capacitator_0805_10uF_X5R -> Capacitator_0603_10uF_X5R; footprint Passive:C_0805 -> Passive:C_0603; symbol Passive:Capacitator_0805_10uF_X5R -> Passive:Capacitator_0603_10uF_X5R; Manufacturer SAMSUNG -> Murata; ManufacturerPartNo CL21A106KOQNNNG -> GRM188R61A106KE69D; Supplier LOM-82-08-32;TME-0805YD106KAT2A;TME-CL21A106KOQNNNG; FAR-12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 -> LOM-82-13-69;
- C4, C5: value Capacitator_0805_22pF_X7R -> Capacitator_0603_22pF_NP0; footprint Passive:C_0805 -> Passive:C_0603; symbol Passive:Capacitator_0805_22pF_X7R -> Passive:Capacitator_0603_22pF_NP0; Manufacturer SAMSUNG -> YAGEO; ManufacturerPartNo CL21C220JBANNNC -> CC0603JRNP09BN220;; Supplier LOM-82-09-18; -> LOM-82-02-18;
- J1: value PinStrip_01x06_Male -> PinHeader_01x06_Male; footprint Connectors:PinStrip_1x06_P2.54mm_Vertical -> Connectors:PinHeader_1x06_P2.54mm_Vertical; symbol Connectors:PinStrip_01x06_Male -> Connectors:PinHeader_01x06_Male; Comment PinStrip_01x06_Male -> PinHeader_01x06_Male
- L2: Comment BLM21A -> 1K00@100MHz
- R1, R12, R6: value Resistor_0805_470R -> Resistor_0603_470R; footprint Passive:R_0805 -> Passive:R_0603; symbol Passive:Resistor_0805_470R -> Passive:Resistor_0603_470R; Manufacturer Walsin -> VIKING; ManufacturerPartNo WR08X471JTL -> WR06X4700FTL; Supplier LOM-81-30-15; -> LOM-80-31-61;TME-CQ0603-470R-1% ;
- R10, R14, R36, R9: value Resistor_0805_10K0 -> Resistor_0603_10K0; footprint Passive:R_0805 -> Passive:R_0603; symbol Passive:Resistor_0805_10K0 -> Passive:Resistor_0603_10K0; Manufacturer Walsin -> ASJ; ManufacturerPartNo WR08X471JTL -> CR16-1002-FK; Supplier LOM-81-30-15; -> LOM-80-15-13;TME-CRCW060310K0FKTABC;
- R11: value Resistor_0805_R_DNP -> Resistor_0603_R_DNP; footprint Passive:R_0805 -> Passive:R_0603; symbol Passive:Resistor_0805_R_DNP -> Passive:Resistor_0603_R_DNP
- R13: value Resistor_0805_0R00 -> Resistor_0603_0R00; footprint Passive:R_0805 -> Passive:R_0603; symbol Passive:Resistor_0805_0R00 -> Passive:Resistor_0603_0R00; Manufacturer VIKING -> Yageo Corp.; ManufacturerPartNo CR-05JL7----0R 0.125W -> RC0603JR-100RL;; Supplier LOM-81-10-02; -> LOM-81-34-80;
- R19, R20, R21, R28, R38, R43: footprint Passive:R_0805 -> Passive:R_0603
- R2, R3, R4: value Resistor_0805_220R -> Resistor_0603_220R; footprint Passive:R_0805 -> Passive:R_0603; symbol Passive:Resistor_0805_220R -> Passive:Resistor_0603_220R; ManufacturerPartNo CR-05FL7--220R 0.125W -> CR-03FL7--220R 0.1W; Supplier LOM-80-10-78; -> LOM-80-11-55;
- R5: value Resistor_0805_4K70 -> Resistor_0603_4K70; footprint Passive:R_0805 -> Passive:R_0603; symbol Passive:Resistor_0805_4K70 -> Passive:Resistor_0603_4K70; Manufacturer VIKING -> ROYAL OHM;; ManufacturerPartNo CR-05FL7---4K7 0.125W -> CQ0603-4K7-1%;; Supplier LOM-80-10-94 -> LOM-80-11-85;TME-CRCW06034K70FKEA;
- U3: value LDO-MCP1700T-3302E_TT-Others -> LDO_MCP1700T-3302E_TT
Connections:
- net +3V3: now also U7.5 (VBAT)
- net +BATT: no longer U7.5 (VBAT)
- net 5V_USB: now also L3.1; no longer J2.1 (VBUS)
- net GNDD: now also J3.1 (Pin_1), J5.1 (Pin_1), Y1.2, Y1.4
- net at C5.1, U1.10 (OSC2): now also Y1.3
- net at C4.1, U1.9 (OSC1): now also Y1.1
- net at F1.2: now also J5.2 (Pin_2); no longer B1.1 (VBAT+)
- net at R15.1, U2.1: now also R16.1; no longer U2.4 (-)
- net at C8.2, R7.2: now also J4.1 (Pin_1)
- net #CH_CPLT renamed CH_CPLT#
- net #DEN renamed DEN#
- net #MCLR renamed MCLR#
- net #PG: no longer names the net of Q3.1 (B), R14.2
- net #PG: now also R45.2; no longer U6.7 (PG#)
- net #PSEN renamed PSEN#
- net #RST: no longer names the net of U7.9 (RES#)
- net #RST: now also R44.2; no longer U1.16 (RB7)
- net DWN renamed DN#
- net OK renamed OK#
- net UP renamed UP#
- new net: J2.1 (VBUS), L3.2
- new net: R16.2, U2.4 (-)
- new net PG#: R45.1, U6.7 (PG#)
- new net RST#: R44.1, U1.16 (RB7)
Other:
- note added: "Battery"
- moved on the sheet: C25, C26, C27, C31, C33, C34, D4, D5, D6, F1, R26, R27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
