File: MLGC210815.sch (KiCad schematic (older format))
At the start: 5 parts

Commit message: update
Parts:
- added D?: LED0805_KP-2012SGC, Passive:R0805, symbol Passive:LED0805_KP-2012SGC
- added R?: R0805_10K0, Passive:R0805, symbol Passive:R0805_10K0
- added R?: R0805_470R, Passive:R0805, symbol Passive:R0805_470R
Connections:
- net labels added: +3.3V
- net labels removed: VCC
- wire segments 9 -> 12
Other:
- moved on the sheet: J?
Changed lines of the file:
@@
 L Processors:PIC32MM0064GPL028-I_SO U?
 U 1 1 6127C052
-P 3400 1650
-F 0 "U?" H 3400 2425 50  0000 C CNN
-F 1 "PIC32MM0064GPL028-I_SO" H 3500 2300 50  0001 C CNN
-F 2 "Integrated Circuits:SOIC-28W" H 3400 800 50  0001 C CNN
-F 3 "..\\KiCad\\Datasheet\\MICROCHIP-PIC32MM0064GPL036.pdf" H 3000 2250 50  0001 C CNN
-F 4 "MICROCHIP" H 3400 1650 50  0001 C CNN "Manufacturer"
-F 5 "PIC32MM0064GPL028-I/SO" H 3400 1650 50  0001 C CNN "ManufacturerPartNo"
-F 6 "FAR-2610365; TME-PIC32MM0064GPL028-I/SO" H 3400 1650 50  0001 C CNN "Supplier"
-F 7 "PIC32MM0064GPL028" H 3400 2334 50  0000 C CNN "Comment"
-	1    3400 1650
+P 3400 2050
+F 0 "U?" H 3400 2825 50  0000 C CNN
+F 1 "PIC32MM0064GPL028-I_SO" H 3500 2700 50  0001 C CNN
+F 2 "Integrated Circuits:SOIC-28W" H 3400 1200 50  0001 C CNN
+F 3 "..\\KiCad\\Datasheet\\MICROCHIP-PIC32MM0064GPL036.pdf" H 3000 2650 50  0001 C CNN
+F 4 "MICROCHIP" H 3400 2050 50  0001 C CNN "Manufacturer"
+F 5 "PIC32MM0064GPL028-I/SO" H 3400 2050 50  0001 C CNN "ManufacturerPartNo"
+F 6 "FAR-2610365; TME-PIC32MM0064GPL028-I/SO" H 3400 2050 50  0001 C CNN "Supplier"
+F 7 "PIC32MM0064GPL028" H 3400 2734 50  0000 C CNN "Comment"
+	1    3400 2050
 	1    0    0    -1
 $EndComp
@@
 L Connectors:PinStrip_01x06_Male J?
 U 1 1 6127D355
-P 750 3000
-F 0 "J?" H 642 2475 50  0000 C CNN
-F 1 "PinStrip_01x06_Male" H 750 2600 50  0001 C CNN
-F 2 "" H 750 3000 50  0001 C CNN
-F 3 "~" H 750 3000 50  0001 C CNN
-F 4 "PinStrip_01x06_Male" H 642 2566 50  0000 C CNN "Comment"
-F 5 "T&T CONNECTION" H 750 3000 50  0001 C CNN "Manufacturer"
-F 6 "PHSS-40-6/3" H 750 3000 50  0001 C CNN "ManufacturerPartNo"
-F 7 "LOM-43-00-73" H 750 3000 50  0001 C CNN "Supplier"
-	1    750  3000
+P 750 3400
+F 0 "J?" H 642 2875 50  0000 C CNN
+F 1 "PinStrip_01x06_Male" H 750 3000 50  0001 C CNN
+F 2 "" H 750 3400 50  0001 C CNN
+F 3 "~" H 750 3400 50  0001 C CNN
+F 4 "PinStrip_01x06_Male" H 642 2966 50  0000 C CNN "Comment"
+F 5 "T&T CONNECTION" H 750 3400 50  0001 C CNN "Manufacturer"
+F 6 "PHSS-40-6/3" H 750 3400 50  0001 C CNN "ManufacturerPartNo"
+F 7 "LOM-43-00-73" H 750 3400 50  0001 C CNN "Supplier"
+	1    750  3400
 	-1   0    0    1
 $EndComp
@@
 L Passive:R0805_220R R?
 U 1 1 61282922
-P 1250 2900
-F 0 "R?" V 1135 2900 50  0000 C CNN
-F 1 "R0805_220R" H 1250 2900 50  0001 C CNN
-F 2 "Passive:R0805" H 1250 2900 50  0001 C CNN
-F 3 "" H 1250 2900 50  0001 C CNN
-F 4 "220R" V 1134 2900 50  0001 C CNN "Comment"
-F 5 "Viking Tech Corp." H 1250 2900 50  0001 C CNN "Manufacturer"
-F 6 "CR-05FL7--220R 0.125W " H 1250 2900 50  0001 C CNN "ManufacturerPartNo"
-F 7 "LOM-80-10-78;" H 1250 2900 50  0001 C CNN "Supplier"
-	1    1250 2900
+P 1250 3300
+F 0 "R?" V 1250 3250 50  0000 C CNN
+F 1 "R0805_220R" H 1250 3300 50  0001 C CNN
+F 2 "Passive:R0805" H 1250 3300 50  0001 C CNN
+F 3 "" H 1250 3300 50  0001 C CNN
+F 4 "220R" V 1134 3300 50  0001 C CNN "Comment"
+F 5 "Viking Tech Corp." H 1250 3300 50  0001 C CNN "Manufacturer"
+F 6 "CR-05FL7--220R 0.125W " H 1250 3300 50  0001 C CNN "ManufacturerPartNo"
+F 7 "LOM-80-10-78;" H 1250 3300 50  0001 C CNN "Supplier"
+	1    1250 3300
 	0    1    1    0
 $EndComp
@@
 L Passive:R0805_220R R?
 U 1 1 61283D40
-P 1250 2800
-F 0 "R?" V 1043 2800 50  0000 C CNN
-F 1 "R0805_220R" H 1250 2800 50  0001 C CNN
-F 2 "Passive:R0805" H 1250 2800 50  0001 C CNN
-F 3 "" H 1250 2800 50  0001 C CNN
-F 4 "220R" V 1134 2800 50  0000 C CNN "Comment"
-F 5 "Viking Tech Corp." H 1250 2800 50  0001 C CNN "Manufacturer"
-F 6 "CR-05FL7--220R 0.125W " H 1250 2800 50  0001 C CNN "ManufacturerPartNo"
-F 7 "LOM-80-10-78;" H 1250 2800 50  0001 C CNN "Supplier"
-	1    1250 2800
-	0    1    1    0
-$EndComp
-$Comp
-L Passive:R0805_220R R?
-U 1 1 61285E48
 P 1250 3200
-F 0 "R?" V 1135 3200 50  0000 C CNN
+F 0 "R?" V 1250 3150 50  0000 C CNN
 F 1 "R0805_220R" H 1250 3200 50  0001 C CNN
 F 2 "Passive:R0805" H 1250 3200 50  0001 C CNN
 F 3 "" H 1250 3200 50  0001 C CNN
-F 4 "220R" V 1134 3200 50  0001 C CNN "Comment"
+F 4 "220R" V 1134 3200 50  0000 C CNN "Comment"
 F 5 "Viking Tech Corp." H 1250 3200 50  0001 C CNN "Manufacturer"
 F 6 "CR-05FL7--220R 0.125W " H 1250 3200 50  0001 C CNN "ManufacturerPartNo"
@@
 	0    1    1    0
 $EndComp
+$Comp
+L Passive:R0805_220R R?
+U 1 1 61285E48
+P 1250 3600
+F 0 "R?" V 1250 3550 50  0000 C CNN
+F 1 "R0805_220R" H 1250 3600 50  0001 C CNN
+F 2 "Passive:R0805" H 1250 3600 50  0001 C CNN
+F 3 "" H 1250 3600 50  0001 C CNN
+F 4 "220R" V 1134 3600 50  0001 C CNN "Comment"
+F 5 "Viking Tech Corp." H 1250 3600 50  0001 C CNN "Manufacturer"
+F 6 "CR-05FL7--220R 0.125W " H 1250 3600 50  0001 C CNN "ManufacturerPartNo"
+F 7 "LOM-80-10-78;" H 1250 3600 50  0001 C CNN "Supplier"
+	1    1250 3600
+	0    1    1    0
+$EndComp
+Wire Wire Line
+	950  3600 1100 3600
+Wire Wire Line
+	950  3300 1100 3300
 Wire Wire Line
 	950  3200 1100 3200
-Wire Wire Line
-	950  2900 1100 2900
-Wire Wire Line
-	950  2800 1100 2800
 $Comp
 L power:GND #PWR?
 U 1 1 6128743A
-P 950 3100
-F 0 "#PWR?" H 950 2850 50  0001 C CNN
-F 1 "GND" V 955 2972 50  0000 R CNN
-F 2 "" H 950 3100 50  0001 C CNN
-F 3 "" H 950 3100 50  0001 C CNN
-	1    950  3100
+P 950 3500
+F 0 "#PWR?" H 950 3250 50  0001 C CNN
+F 1 "GND" V 955 3372 50  0000 R CNN
+F 2 "" H 950 3500 50  0001 C CNN
+F 3 "" H 950 3500 50  0001 C CNN
+	1    950  3500
 	0    -1   -1   0
 $EndComp
-$Comp
-L power:VCC #PWR?
-U 1 1 612887AD
-P 950 3000
-F 0 "#PWR?" H 950 2850 50  0001 C CNN
-F 1 "VCC" V 965 3128 50  0000 L CNN
-F 2 "" H 950 3000 50  0001 C CNN
-F 3 "" H 950 3000 50  0001 C CNN
-	1    950  3000
-	0    1    1    0
-$EndComp
-Wire Wire Line
-	1800 3200 1400 3200
-Text Label 1400 2800 0    50   ~ 0
+Text Label 1400 3200 0    50   ~ 0
 PGC-RB6
-Text Label 1400 2900 0    50   ~ 0
+Text Label 1400 3300 0    50   ~ 0
 PGD-RB7
-Text Label 1400 3200 0    50   ~ 0
+Text Label 1400 3600 0    50   ~ 0
 #MCLR
 Wire Wire Line
-	3850 2400 3850 2800
-Wire Wire Line
-	1400 2800 3850 2800
-Wire Wire Line
-	3950 2900 3950 2300
-Wire Wire Line
-	1400 2900 3950 2900
-Wire Wire Line
-	3850 2300 3950 2300
+	3850 2800 3850 3200
+Wire Wire Line
+	1400 3200 3850 3200
+Wire Wire Line
+	3950 3300 3950 2700
+Wire Wire Line
+	1400 3300 3950 3300
+Wire Wire Line
+	3850 2700 3950 2700
+$Comp
+L Passive:R0805_10K0 R?
+U 1 1 6127F021
+P 2650 1350
+F 0 "R?" H 2720 1396 50  0000 L CNN
+F 1 "R0805_10K0" H 2650 1350 50  0001 C CNN
+F 2 "Passive:R0805" H 2650 1350 50  0001 C CNN
+F 3 "" H 2650 1350 50  0001 C CNN
+F 4 "10K0" H 2720 1305 50  0000 L CNN "Comment"
+F 5 "Walsin" H 2650 1350 50  0001 C CNN "Manufacturer"
+F 6 "WR08X471JTL" H 2650 1350 50  0001 C CNN "ManufacturerPartNo"
+F 7 "LOM-81-30-15;" H 2650 1350 50  0001 C CNN "Supplier"
+	1    2650 1350
+	1    0    0    -1
+$EndComp
+Wire Wire Line
+	2950 1500 2650 1500
+Wire Wire Line
+	2650 1500 2650 3600
+Wire Wire Line
+	1400 3600 2650 3600
+Connection ~ 2650 1500
+$Comp
+L power:+3.3V #PWR?
+U 1 1 6128026D
+P 2650 1200
+F 0 "#PWR?" H 2650 1050 50  0001 C CNN
+F 1 "+3.3V" H 2665 1373 50  0000 C CNN
+F 2 "" H 2650 1200 50  0001 C CNN
+F 3 "" H 2650 1200 50  0001 C CNN
+	1    2650 1200
+	1    0    0    -1
+$EndComp
+$Comp
+L power:+3.3V #PWR?
+U 1 1 61280D20
+P 950 3400
+F 0 "#PWR?" H 950 3250 50  0001 C CNN
+F 1 "+3.3V" V 965 3528 50  0000 L CNN
+F 2 "" H 950 3400 50  0001 C CNN
+F 3 "" H 950 3400 50  0001 C CNN
+	1    950  3400
+	0    1    1    0
+$EndComp
+$Comp
+L Passive:LED0805_KP-2012SGC D?
+U 1 1 61289879
+P 850 4150
+F 0 "D?" V 889 4032 50  0000 R CNN
+F 1 "LED0805_KP-2012SGC" H 850 4150 50  0001 C CNN
+F 2 "Passive:R0805" H 850 4150 50  0001 C CNN
+F 3 "" H 850 4150 50  0001 C CNN
+F 4 "Green" V 798 4032 50  0000 R CNN "Comment"
+F 5 "KINGBRIGHT" H 850 4150 50  0001 C CNN "Manufacturer"
+F 6 "KP-2010SGC" H 850 4150 50  0001 C CNN "ManufacturerPartNo"
+F 7 "TME-KP-2012SGC;FAR-2099239;LOM-95-01-09" H 850 4150 50  0001 C CNN "Supplier"
+	1    850  4150
+	0    -1   -1   0
+$EndComp
+$Comp
+L Passive:R0805_470R R?
+U 1 1 6128B060
+P 850 4500
+F 0 "R?" V 643 4500 50  0000 C CNN
+F 1 "R0805_470R" H 850 4500 50  0001 C CNN
+F 2 "Passive:R0805" H 850 4500 50  0001 C CNN
+F 3 "" H 850 4500 50  0001 C CNN
+F 4 "470R" V 734 4500 50  0000 C CNN "Comment"
+F 5 "Walsin" H 850 4500 50  0001 C CNN "Manufacturer"
+F 6 "WR08X471JTL" H 850 4500 50  0001 C CNN "ManufacturerPartNo"
+F 7 "LOM-81-30-15;" H 850 4500 50  0001 C CNN "Supplier"
+	1    850  4500
+	1    0    0    -1
+$EndComp
+$Comp
+L power:GND #PWR?
+U 1 1 6128BDFB
+P 850 4650
+F 0 "#PWR?" H 850 4400 50  0001 C CNN
+F 1 "GND" V 855 4522 50  0000 R CNN
+F 2 "" H 850 4650 50  0001 C CNN
+F 3 "" H 850 4650 50  0001 C CNN
+	1    850  4650
+	1    0    0    -1
+$EndComp
+$Comp
+L power:+3.3V #PWR?
+U 1 1 6128CA37
+P 850 4000
+F 0 "#PWR?" H 850 3850 50  0001 C CNN
+F 1 "+3.3V" H 865 4173 50  0000 C CNN
+F 2 "" H 850 4000 50  0001 C CNN
+F 3 "" H 850 4000 50  0001 C CNN
+	1    850  4000
+	1    0    0    -1
+$EndComp
+Wire Wire Line
+	850  4300 850  4350
 $EndSCHEMATC

Commit message: update
Parts:
- J1: renamed from J?; footprint (none) -> Connectors:PinStrip_1x06_P2.54mm_Vertical
- gave numbers to parts that had none: 7
Changed lines of the file:
@@
 $EndDescr
 $Comp
-L Processors:PIC32MM0064GPL028-I_SO U?
+L Processors:PIC32MM0064GPL028-I_SO U1
 U 1 1 6127C052
 P 3400 2050
-F 0 "U?" H 3400 2825 50  0000 C CNN
+F 0 "U1" H 3400 2825 50  0000 C CNN
 F 1 "PIC32MM0064GPL028-I_SO" H 3500 2700 50  0001 C CNN
 F 2 "Integrated Circuits:SOIC-28W" H 3400 1200 50  0001 C CNN
@@
 $EndComp
 $Comp
-L Connectors:PinStrip_01x06_Male J?
+L Connectors:PinStrip_01x06_Male J1
 U 1 1 6127D355
 P 750 3400
-F 0 "J?" H 642 2875 50  0000 C CNN
+F 0 "J1" H 642 2875 50  0000 C CNN
 F 1 "PinStrip_01x06_Male" H 750 3000 50  0001 C CNN
-F 2 "" H 750 3400 50  0001 C CNN
+F 2 "Connectors:PinStrip_1x06_P2.54mm_Vertical" H 750 3400 50  0001 C CNN
 F 3 "~" H 750 3400 50  0001 C CNN
 F 4 "PinStrip_01x06_Male" H 642 2966 50  0000 C CNN "Comment"
@@
 $EndComp
 $Comp
-L Passive:R0805_220R R?
+L Passive:R0805_220R R3
 U 1 1 61282922
 P 1250 3300
-F 0 "R?" V 1250 3250 50  0000 C CNN
+F 0 "R3" V 1250 3250 50  0000 C CNN
 F 1 "R0805_220R" H 1250 3300 50  0001 C CNN
 F 2 "Passive:R0805" H 1250 3300 50  0001 C CNN
@@
 $EndComp
 $Comp
-L Passive:R0805_220R R?
+L Passive:R0805_220R R2
 U 1 1 61283D40
 P 1250 3200
-F 0 "R?" V 1250 3150 50  0000 C CNN
+F 0 "R2" V 1250 3150 50  0000 C CNN
 F 1 "R0805_220R" H 1250 3200 50  0001 C CNN
 F 2 "Passive:R0805" H 1250 3200 50  0001 C CNN
@@
 $EndComp
 $Comp
-L Passive:R0805_220R R?
+L Passive:R0805_220R R4
 U 1 1 61285E48
 P 1250 3600
-F 0 "R?" V 1250 3550 50  0000 C CNN
+F 0 "R4" V 1250 3550 50  0000 C CNN
 F 1 "R0805_220R" H 1250 3600 50  0001 C CNN
 F 2 "Passive:R0805" H 1250 3600 50  0001 C CNN
@@
 	950  3200 1100 3200
 $Comp
-L power:GND #PWR?
+L power:GND #PWR04
 U 1 1 6128743A
 P 950 3500
-F 0 "#PWR?" H 950 3250 50  0001 C CNN
+F 0 "#PWR04" H 950 3250 50  0001 C CNN
 F 1 "GND" V 955 3372 50  0000 R CNN
 F 2 "" H 950 3500 50  0001 C CNN
@@
 	3850 2700 3950 2700
 $Comp
-L Passive:R0805_10K0 R?
+L Passive:R0805_10K0 R5
 U 1 1 6127F021
 P 2650 1350
-F 0 "R?" H 2720 1396 50  0000 L CNN
+F 0 "R5" H 2720 1396 50  0000 L CNN
 F 1 "R0805_10K0" H 2650 1350 50  0001 C CNN
 F 2 "Passive:R0805" H 2650 1350 50  0001 C CNN
@@
 Connection ~ 2650 1500
 $Comp
-L power:+3.3V #PWR?
+L power:+3.3V #PWR05
 U 1 1 6128026D
 P 2650 1200
-F 0 "#PWR?" H 2650 1050 50  0001 C CNN
+F 0 "#PWR05" H 2650 1050 50  0001 C CNN
 F 1 "+3.3V" H 2665 1373 50  0000 C CNN
 F 2 "" H 2650 1200 50  0001 C CNN
@@
 $EndComp
 $Comp
-L power:+3.3V #PWR?
+L power:+3.3V #PWR03
 U 1 1 61280D20
 P 950 3400
-F 0 "#PWR?" H 950 3250 50  0001 C CNN
+F 0 "#PWR03" H 950 3250 50  0001 C CNN
 F 1 "+3.3V" V 965 3528 50  0000 L CNN
 F 2 "" H 950 3400 50  0001 C CNN
@@
 $EndComp
 $Comp
-L Passive:LED0805_KP-2012SGC D?
+L Passive:LED0805_KP-2012SGC D1
 U 1 1 61289879
 P 850 4150
-F 0 "D?" V 889 4032 50  0000 R CNN
+F 0 "D1" V 889 4032 50  0000 R CNN
 F 1 "LED0805_KP-2012SGC" H 850 4150 50  0001 C CNN
 F 2 "Passive:R0805" H 850 4150 50  0001 C CNN
@@
 $EndComp
 $Comp
-L Passive:R0805_470R R?
+L Passive:R0805_470R R1
 U 1 1 6128B060
 P 850 4500
-F 0 "R?" V 643 4500 50  0000 C CNN
+F 0 "R1" V 643 4500 50  0000 C CNN
 F 1 "R0805_470R" H 850 4500 50  0001 C CNN
 F 2 "Passive:R0805" H 850 4500 50  0001 C CNN
@@
 $EndComp
 $Comp
-L power:GND #PWR?
+L power:GND #PWR02
 U 1 1 6128BDFB
 P 850 4650
-F 0 "#PWR?" H 850 4400 50  0001 C CNN
+F 0 "#PWR02" H 850 4400 50  0001 C CNN
 F 1 "GND" V 855 4522 50  0000 R CNN
 F 2 "" H 850 4650 50  0001 C CNN
@@
 $EndComp
 $Comp
-L power:+3.3V #PWR?
+L power:+3.3V #PWR01
 U 1 1 6128CA37
 P 850 4000
-F 0 "#PWR?" H 850 3850 50  0001 C CNN
+F 0 "#PWR01" H 850 3850 50  0001 C CNN
 F 1 "+3.3V" H 865 4173 50  0000 C CNN
 F 2 "" H 850 4000 50  0001 C CNN

Commit message: update
Parts:
- removed R5: R0805_10K0, Passive:R0805, symbol Passive:R0805_10K0
- removed U1: PIC32MM0064GPL028-I_SO, Integrated Circuits:SOIC-28W, symbol Processors:PIC32MM0064GPL028-I_SO
- added B1: L402036, Others:Battery_L402036, symbol Others:L402036
- added C1, C2: C0805_100nF, Passive:C0805, symbol Passive:C0805_100nF
- added C3: C0805_10uF, Passive:C0805, symbol Passive:C0805_10uF
- added C? (x4): C0805_1uF_X7R, Passive:C0805, symbol Passive:C0805_1uF_X7R
- added J?: USB-B-04PFHTW, symbol Connectors:USB-B-04PFHTW
- added Q?: BC817, Package_TO_SOT_SMD:SOT-23, symbol Others:BC817
- added R5: R0805_4K70, Passive:R0805, symbol Passive:R0805_4K70
- added U1: PIC32MX170F256B-ISS, Integrated Circuits:SSOP-28, symbol Processors:PIC32MX170F256B-ISS
- added U2: RX1602A5-BIW-TS, symbol Others:RX1602A5-BIW-TS
- added U?: MCP73833-FCI_UN, symbol Others:MCP73833-FCI_UN
- added U?: MCP1700T-3302E_TT, Package_TO_SOT_SMD:SOT-23, symbol Others:MCP1700T-3302E_TT
Connections:
- net labels added: GNDD, IC1, PGC, PGD, SCL, SDA
- net labels removed: PGC-RB6, PGD-RB7
- wire segments 12 -> 51
Other:
- note added: "BK: min 3.4V, max 3.6V"
- note added: "Vin:2.3V..3.6V"
- note added: "Vout: 2.75V..4.2V"
- note added: "fuse"
- note added: "switch"
- moved on the sheet: J1

Commit message: update
Parts:
- removed C? (x2): C0805_1uF_X7R, Passive:C0805, symbol Passive:C0805_1uF_X7R
- removed U2: RX1602A5-BIW-TS, symbol Others:RX1602A5-BIW-TS
- added C? (x2): C0805_22pF_X7R, Passive:C0805, symbol Passive:Capacitator_0805_22pF_X7R
- added C? (x2): Capacitator_0805_100nF_X7R, Passive:C0805, symbol Passive:Capacitator_0805_100nF_X7R
- added C? (x2): Capacitator_0603_2.2uF_X5R, Passive:C0603, symbol Passive:Capacitator_0603_2.2uF_X5R
- added C? (x3): Capacitator_0603_100nF_X7R, Passive:C0603, symbol Passive:Capacitator_0603_100nF_X7R
- added C? (x2): Capacitator_0603_47pF_X7R, Passive:C0603, symbol Passive:Capacitator_0603_47pF_X7R
- added D? (x2): LED0805_KP-2012SGC, Passive:R0805, symbol MLGC210815-rescue:LED0805_KP-2012SGC-Passive
- added F?: Polyfuse_1812_1100mA_33V, symbol Passive:Polyfuse_1812_1100mA_33V
- added L?: Inductor_0805_10uH, symbol Passive:Inductor_0805_10uH
- added Q?: P-MOSFET-SI2315BDS-T1-E3, symbol Others:P-MOSFET-SI2315BDS-T1-E3
- added R?: Resistor_0805_0R00, Passive:R0805, symbol Passive:Resistor_0805_0R00
- added R? (x3): Resistor_0805_R_DNP, Passive:R0805, symbol Passive:Resistor_0805_R_DNP
- added R? (x2): Resistor_0805_10K0, Passive:R0805, symbol Passive:Resistor_0805_10K0
- added R?: Resistor_0805_470R, Passive:R0805, symbol Passive:Resistor_0805_470R
- added R? (x3): Resistor_0603_220R, Passive:R0603, symbol Passive:Resistor_0603_220R
- added R? (x2): Resistor_0603_27R0, Passive:R0603, symbol Passive:Resistor_0603_27R0
- added R? (x2): Resistor_0603_470R, Passive:R0805, symbol Passive:Resistor_0603_470R
- added U?: DISPLAY-REX012832FSPP3N01, symbol Others:DISPLAY-REX012832FSPP3N01
- added U?: OPA-MCP6V36T-E_OT, symbol Others:OPA-MCP6V36T-E_OT
- added U?: SENSOR-BMA250E, symbol Others:SENSOR-BMA250E
- added U?: Interface-FT230XS, Package_SO:SSOP-16_3.9x4.9mm_P0.635mm, symbol Others:Interface-FT230XS
- added Y?: HC49SM_8MHz, symbol Passive:Crystal_HC49SM_8MHz
- B1: symbol Others:L402036 -> Others:BATTERY-L402036
- C1, C2: symbol Passive:C0805_100nF -> Passive:Capacitator_0805_100nF_X7R
- C3: symbol Passive:C0805_10uF -> Passive:Capacitator_0805_10uF_X5R
- C? (x2): symbol Passive:C0805_1uF_X7R -> Passive:Capacitator_0805_1uF_X7R
- D1: symbol Passive:LED0805_KP-2012SGC -> MLGC210815-rescue:LED0805_KP-2012SGC-Passive
- Q?: symbol Others:BC817 -> Others:NPN-BC817
- R1: symbol Passive:R0805_470R -> Passive:Resistor_0805_470R
- R2, R3, R4: symbol Passive:R0805_220R -> Passive:Resistor_0805_220R
- R5: symbol Passive:R0805_4K70 -> Passive:Resistor_0805_4K70
- U?: symbol Others:MCP73833-FCI_UN -> Others:BATTERY-MCP73833-FCI_UN
- U?: symbol Others:MCP1700T-3302E_TT -> Others:LDO-MCP1700T-3302E_TT
Connections:
- net labels added: #PSEN, +3V3_USB, +BATT, 5V_USB, AN0, D+, D-, INT1, PC-RX, PC-TX, SCL1, SDA1, U1RX, U1TX, VDDA
- net labels removed: GND, SCL, SDA
- wire segments 51 -> 144
- no-connect marks 0 -> 6
Other:
- note added: "51K0/16K0"
- note added: "5V->1.2V"
- note added: "ADC VREF:1.2V"
- note added: "LQM21FN100N00L"
- note added: "MLF2012E100KT"
- note added: "PICKit"
- moved on the sheet: J1, J?

Commit message: update
Parts:
- removed R? (x2): Resistor_0805_R_DNP, Passive:R0805, symbol Passive:Resistor_0805_R_DNP
- added C? (x5): Capacitator_0805_1uF_X7R, Passive:C0603, symbol Passive:Capacitator_0805_1uF_X7R
- added C? (x3): Capacitator_0603_2.2uF_X5R, Passive:C0603, symbol Passive:Capacitator_0603_2.2uF_X5R
- added C? (x2): C0805_100nF, Passive:C0805, symbol Passive:Capacitator_0805_100nF_X7R
- added C? (x3): Capacitator_0603_47nF_X7R, Passive:C0603, symbol Passive:Capacitator_0603_47nF_X7R
- added C? (x4): Capacitator_0603_100nF_X7R, Passive:C0603, symbol Passive:Capacitator_0603_100nF_X7R
- added C? (x3): Capacitator_0603_1nF_NP0, Passive:C0603, symbol Passive:Capacitator_0603_1nF_NP0
- added D?: LED_0603_Blue, Passive:R0603, symbol Passive:LED_0603_Blue
- added D?: LED0805_KP-2012SGC, Passive:R0805, symbol MLGC210815-rescue:LED0805_KP-2012SGC-Passive
- added D?: DIODE-BAT54S, symbol Others:DIODE-BAT54S
- added L?: Filter_0805_BLM21A102SPT, symbol Passive:Filter_0805_BLM21A102SPT
- added Q?: P-MOSFET-SI2315BDS-T1-E3, symbol Others:P-MOSFET-SI2315BDS-T1-E3
- added Q?: BC817, Package_TO_SOT_SMD:SOT-23, symbol Others:NPN-BC817
- added R?: Resistor_0603_0R00, Passive:R0603, symbol Passive:Resistor_0603_0R00
- added R?: Resistor_0603_150K, Passive:R0603, symbol Passive:Resistor_0603_150K
- added R? (x2): Resistor_0805_10K0, Passive:R0805, symbol Passive:Resistor_0805_10K0
- added R?: Resistor_0603_R_DNP, Passive:R0603, symbol Passive:Resistor_0603_R_DNP
- added R?: Resistor_0603_1K00, Passive:R0603, symbol Passive:Resistor_0603_1K00
- added R? (x4): Resistor_0603_10K0, Passive:R0805, symbol Passive:Resistor_0603_10K0
- added R?: Resistor_0603_150K, Passive:R0603, symbol Passive:Resistor_0603_39K0
- added R? (x8): Resistor_0603_4K70, Passive:R0603, symbol Passive:Resistor_0603_4K70
- added R?: Resistor_0603_13K0, Passive:R0603, symbol Passive:Resistor_0603_11K0
- added R? (x3): Resistor_0603_10R0, Passive:R0603, symbol Passive:Resistor_0603_10R0
- added R?: Resistor_0805_470R, Passive:R0805, symbol Passive:Resistor_0805_470R
- added R? (x2): Resistor_0603_9K10, Passive:R0603, symbol Passive:Resistor_0603_9K10
- added SW? (x3): Switch_Tact_OMRON-B3F-3100, symbol Others:Switch_Tact_OMRON-B3F-3100
- added TH?: NTC_0603_10K, symbol Passive:NTC_0603_10K
Connections:
- net labels added: #CH_CPLT, #DEN, #PG, #RST, +3.3VA, AN1, DWN, LIVE_LED, OK, UP
- net labels removed: VDDA
- wire segments 144 -> 235
- no-connect marks 6 -> 9
Other:
- note added: "15V->3.3V\n3900/1100"
- note added: "5V->3.3V\n4700/9100"
- note added: "OC?"
- note added: "PG LOW = MCLR HIGH\nPG HIGH = MCLR LOW"
- note added: "VREF:AVDD"
- note removed: "51K0/16K0"
- note removed: "5V->1.2V"
- note removed: "ADC VREF:1.2V"
- note removed: "BK: min 3.4V, max 3.6V"
- note removed: "LQM21FN100N00L"
- note removed: "MLF2012E100KT"
- note removed: "fuse"
- note removed: "switch"
- moved on the sheet: B1, C1, C2, C3, C?, D1, D?, F?, J1, J?, L?, Q?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

Commit message: update
Parts:
- added R44: Resistor_0603_0R00, Passive:R0603, symbol Passive:Resistor_0603_0R00
- B1: footprint Others:Battery_L402036 -> Others:CELLEVIA_L402036; symbol Others:BATTERY-L402036 -> MLGC210815-rescue:BATTERY_CELLEVIA-L402036-Others
- C26, C34: renamed from C?; footprint Passive:C0805 -> Passive:C0603; Manufacturer YAGEO; SAMSUNG; -> YAGEO;; ManufacturerPartNo CC0805KKX7R7BB105;CL21B105KBFNNNG; -> CC0603KRX7R7BB105; Supplier LOM-82-05-11;FAR-2370711;TME-CC0805KKX7R7BB105; -> LOM-82-06-80;TME-CC0603KRX7R7105;
- D2: renamed from D?; symbol Others:DIODE-BAT54S -> MLGC210815-rescue:DIODE-BAT54S-Others
- J2: renamed from J?; footprint (none) -> Connectors:T-T_USB-B-04PFHTW
- Q1: renamed from Q?; symbol Others:P-MOSFET-SI2315BDS-T1-E3 -> MLGC210815-rescue:P-MOSFET-SI2315BDS-T1-E3-Others
- Q2: renamed from Q?; footprint Package_TO_SOT_SMD:SOT-23 -> Semiconductor:SOT-23; symbol Others:NPN-BC817 -> Others:NPN_BC817; Comment BC817-25LT1G -> BC817
- Q3: renamed from Q?; footprint Package_TO_SOT_SMD:SOT-23 -> Semiconductor:SOT-23; symbol Others:NPN-BC817 -> Others:NPN_BC817
- Q4: renamed from Q?; footprint (none) -> Semiconductor:SOT-23; symbol Others:P-MOSFET-SI2315BDS-T1-E3 -> Others:P-MOSFET_SI2315BDS-T1-E3
- SW1, SW2, SW3: renamed from SW?; symbol Others:Switch_Tact_OMRON-B3F-3100 -> MLGC210815-rescue:Switch_Tact_OMRON-B3F-3100-Others
- U1: footprint Integrated Circuits:SSOP-28 -> Semiconductor:SSOP-28
- U2: renamed from U?; footprint (none) -> Semiconductor:SOT-23-5; symbol Others:OPA-MCP6V36T-E_OT -> Others:OPA_MCP6V36T-E_OT
- U3: renamed from U?; symbol Others:LDO-MCP1700T-3302E_TT -> MLGC210815-rescue:LDO-MCP1700T-3302E_TT-Others
- U4: renamed from U?; footprint (none) -> Semiconductor:LGA-12; symbol Others:SENSOR-BMA250E -> Others:SENSOR_BMA250E
- U5: renamed from U?; footprint Package_SO:SSOP-16_3.9x4.9mm_P0.635mm -> Semiconductor:SSOP-16; symbol Others:Interface-FT230XS -> Others:INTERFACE_FT230XS
- U6: renamed from U?; footprint (none) -> Integrated Circuits:MSOP-10; symbol Others:BATTERY-MCP73833-FCI_UN -> Others:BATTERY_MCP73833-FCI_UN
- U7: renamed from U?; footprint (none) -> Others:RAYSTAR_REX012832; symbol Others:DISPLAY-REX012832FSPP3N01 -> Others:DISPLAY_REX012832FSPP3N01
- gave numbers to parts that had none: 78
Connections:
- net +3V3: now also U4.7 (VDD); no longer U4.4 (VDD)
- net +BATT: now also C12.1, R16.1, U3.3 (VI)
- net GNDD: now also R44.1; no longer B1.2 (VBAT-)
- net INT1: now also U1.7 (RB3)
- new net: B1.2 (VBAT-), R44.2
- no-connect marks 9 -> 7
Other:
- moved on the sheet: B1
