File: _autosave-MLGC210815.kicad_pcb (KiCad board)
At the start: 2 copper layers, 95 x 24 mm, 110 parts, among them J1 PinHeader_01x06_Male, J2 USB-B-04PFHTW, J3 PinHeader_01x01_Male, J4 PinHeader_01x01_Male, J5 PinHeader_01x02_Male, Q1 P-MOSFET_SI2315BDS-T1-E3, Q2 NPN_BC817, Q3 NPN_BC817, Q4 P-MOSFET_SI2315BDS-T1-E3, SW1 Switch-Tact_OMRON-B3F-3100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

Commit message: update
Parts:
- moved B1 32.2 mm to (62.7, -13.5)
- moved Q2 0.51 mm to (10.2, -13.7)
Routing:
- net +3.3VA: track 39.0 -> 40.5 mm
- net GNDD: track 159.3 -> 158.5 mm
- net Net-(C11-Pad2): track 7.98 -> 8.70 mm
- added copper zone on B.Cu, net Net-(C8-Pad2)
Other:
- board text added: "MLGC210815V00"
