File: _autosave-MLGC210815.kicad_pcb (KiCad board)
At the start: 2 copper layers, 95 x 24 mm, 110 parts, among them J1 PinHeader_01x06_Male, J2 USB-B-04PFHTW, J3 PinHeader_01x01_Male, J4 PinHeader_01x01_Male, J5 PinHeader_01x02_Male, Q1 P-MOSFET_SI2315BDS-T1-E3, Q2 NPN_BC817, Q3 NPN_BC817, Q4 P-MOSFET_SI2315BDS-T1-E3, SW1 Switch-Tact_OMRON-B3F-3100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

Commit message: update
Connections:
- U4 pad 4: Net-(U4-Pad4) -> GNDD
Routing:
- net /D+: track 15.9 -> 13.3 mm
