File: MLGC210815.kicad_pcb (KiCad board)
At the start: 2 copper layers, 8 parts, among them J1 PinStrip_01x06_Male, U1 PIC32MM0064GPL028-I_SO

Commit message: update
Parts:
- added B1: L402036, Others:Battery_L402036, F.Cu at (143.5, 70.5)
- added C1: C0805_100nF, Passive:C0805, F.Cu at (113.5, 72.8)
- added C2: C0805_100nF, Passive:C0805, F.Cu at (156.2, 86.4)
- added C3: C0805_10uF, Passive:C0805, F.Cu at (117.9, 72.8)
- added R5: R0805_4K70, Passive:R0805, F.Cu at (113.5, 75.8)
- U1: value PIC32MM0064GPL028-I_SO -> PIC32MX170F256B-ISS; footprint Integrated Circuits:SOIC-28W -> Integrated Circuits:SSOP-28
- moved J1 35.5 mm to (128.9, 90.8), turned to 90 degrees
- moved R3 20.7 mm to (134.0, 87.0), turned to 0 degrees
- moved R2 15.4 mm to (137.8, 87.0), turned to 0 degrees
- moved U1 1.42 mm to (135.3, 78.7)
- moved D1 1.27 mm to (151.1, 83.8)
Connections:
- net Net-(U1-Pad17) renamed /SCL
- net Net-(U1-Pad6) renamed /IC1
- J1 pad 2: GND -> +3V3
- J1 pad 3: +3V3 -> GND
- R2 pad 1: /PGC-RB6 -> /PGC
- R3 pad 1: /PGD-RB7 -> /PGD
- U1 pad 13: Net-(U1-Pad13) -> +3V3
- U1 pad 15: /PGC-RB6 -> Net-(U1-Pad15)
- U1 pad 16: /PGD-RB7 -> /SDA
- U1 pad 27: Net-(U1-Pad27) -> GND
- U1 pad 28: Net-(U1-Pad28) -> +3V3
- U1 pad 4: Net-(U1-Pad4) -> /PGD
- U1 pad 5: Net-(U1-Pad5) -> /PGC
- U1 pad 8: Net-(U1-Pad8) -> GND
Routing:
- net Net-(J1-Pad6): track 0.00 -> 27.3 mm, vias 0 -> 3
- net /PGD: track 0.00 -> 21.0 mm, vias 0 -> 1
- net /PGC: track 0.00 -> 17.3 mm
- net Net-(J1-Pad4): track 0.00 -> 5.02 mm
- net Net-(J1-Pad5): track 0.00 -> 3.86 mm
- net Net-(D1-Pad1): track 0.00 -> 2.79 mm
Other:
- board outline added: 88.9 x 23.5 mm

Commit message: updATE
Parts:
- removed the R5 at (121.9, 83.8)
- added C10: Capacitator_0805_100nF_X7R, Passive:C_0805, F.Cu at (245.1, 85.9)
- added C11: Capacitator_0805_100nF_X7R, Passive:C_0805, F.Cu at (227.3, 101.0)
- added C12: Capacitator_0805_1uF_X7R, Passive:C_0603, F.Cu at (223.0, 112.9)
- added C13: Capacitator_0603_47nF_X7R, Passive:C_0603, F.Cu at (231.9, 103.2)
- added C14: Capacitator_0603_47nF_X7R, Passive:C_0603, F.Cu at (239.1, 97.3)
- added C15: Capacitator_0603_100nF_X7R, Passive:C_0603, F.Cu at (249.3, 88.7)
- added C16: Capacitator_0805_1uF_X7R, Passive:C_0603, F.Cu at (231.9, 105.7)
- added C17: Capacitator_0603_100nF_X7R, Passive:C_0603, F.Cu at (226.4, 121.8)
- added C18: Capacitator_0603_100nF_X7R, Passive:C_0603, F.Cu at (227.2, 119.3)
- added C19: Capacitator_0603_100nF_X7R, Passive:C_0603, F.Cu at (239.9, 107.4)
- added C20: Capacitator_0603_1nF_NP0, Passive:C_0603, F.Cu at (231.2, 115.8)
- added C21: Capacitator_0603_1nF_NP0, Passive:C_0603, F.Cu at (248.0, 99.3)
- added C22: Capacitator_0603_1nF_NP0, Passive:C_0603, F.Cu at (251.6, 96.7)
- added C23: Capacitator_0603_100nF_X7R, Passive:C_0603, F.Cu at (244.0, 104.4)
- added C24: Capacitator_0603_100nF_X7R, Passive:C_0603, F.Cu at (248.0, 101.8)
- added C25: Capacitator_0603_47nF_X7R, Passive:C_0603, F.Cu at (231.2, 118.3)
- added C26: Capacitator_0805_1uF_X7R, Passive:C_0603, F.Cu at (239.5, 109.9)
- added C27: Capacitator_0603_100nF_X7R, Passive:C_0603, F.Cu at (235.5, 110.7)
- added C28: Capacitator_0603_2.2uF_X5R, Passive:C_0603, F.Cu at (227.5, 109.3)
- added C29: Capacitator_0603_2.2uF_X5R, Passive:C_0603, F.Cu at (231.5, 108.2)
- added C30: Capacitator_0603_2.2uF_X5R, Passive:C_0603, F.Cu at (218.4, 121.7)
- added C31: Capacitator_0603_47pF_X7R, Passive:C_0603, F.Cu at (243.5, 96.9)
- added C32: Capacitator_0603_2.2uF_X5R, Passive:C_0603, F.Cu at (249.0, 91.7)
- added C33: Capacitator_0603_47pF_X7R, Passive:C_0603, F.Cu at (223.2, 115.4)
- added C34: Capacitator_0805_1uF_X7R, Passive:C_0603, F.Cu at (235.9, 103.2)
- added C35: Capacitator_0805_1uF_X7R, Passive:C_0603, F.Cu at (227.5, 111.8)
- added C36: Capacitator_0805_1uF_X7R, Passive:C_0603, F.Cu at (253.8, 85.7)
- added C4: Capacitator_0805_22pF_X7R, Passive:C_0805, F.Cu at (222.9, 101.0)
- added C5: Capacitator_0805_22pF_X7R, Passive:C_0805, F.Cu at (205.7, 121.4)
- added C6: Capacitator_0805_100nF_X7R, Passive:C_0805, F.Cu at (218.8, 110.2)
- added C7: Capacitator_0603_2.2uF_X5R, Passive:C_0603, F.Cu at (218.4, 119.2)
- added C8: Capacitator_0805_100nF_X7R, Passive:C_0805, F.Cu at (210.1, 116.9)
- added C9: Capacitator_0805_1uF_X7R, Passive:C_0603, F.Cu at (236.0, 100.3)
- added D2: DIODE_BAT54S, Semiconductor:SOT-23, F.Cu at (214.4, 112.7)
- added D3: LED_0603_Green, Passive:LED_0603_GRE, F.Cu at (245.0, 91.7)
- added D4: LED_0603_Green, Passive:LED_0603_GRE, F.Cu at (227.5, 106.7)
- added D5: LED_0603_Green, Passive:LED_0603_GRE, F.Cu at (214.4, 121.8)
- added D6: LED_0603_Blue, Passive:LED_0603_BLU, F.Cu at (214.4, 119.2)
- added F1: Polyfuse_1812_1100mA_33V, Passive:F_1812, F.Cu at (157.5, 71.8)
- added J2: USB-B-04PFHTW, Connectors:T-T_USB-B-04PFHTW, F.Cu at (161.9, 80.0)
- added L1: Inductor_0805_10uH, Passive:L_0805, F.Cu at (196.6, 121.2)
- added L2: Filter_0805_BLM21A102SPT, Passive:L_0805, F.Cu at (201.2, 121.2)
- added Q1: P-MOSFET_SI2315BDS-T1-E3, Semiconductor:SOT-23, F.Cu at (207.4, 113.1)
- added Q2: NPN_BC817, Semiconductor:SOT-23, F.Cu at (230.5, 95.4)
- added Q3: NPN_BC817, Semiconductor:SOT-23, F.Cu at (218.8, 106.4)
- added Q4: P-MOSFET_SI2315BDS-T1-E3, Semiconductor:SOT-23, F.Cu at (205.7, 117.6)
- added R10: Resistor_0805_10K0, Passive:R_0805, F.Cu at (239.3, 94.6)
- added R11: Resistor_0805_R_DNP, Passive:R_0805, F.Cu at (249.6, 85.9)
- added R12: Resistor_0805_470R, Passive:R_0805, F.Cu at (231.8, 100.5)
- added R13: Resistor_0805_0R00, Passive:R_0805, F.Cu at (214.6, 116.4)
- added R14: Resistor_0805_10K0, Passive:R_0805, F.Cu at (218.8, 113.1)
- added R15: Resistor_0603_10R0, Passive:R_0603, F.Cu at (227.2, 114.3)
- added R16: Resistor_0603_4K70, Passive:R_0603, F.Cu at (247.6, 94.2)
- added R17: Resistor_0603_9K10, Passive:R_0603, F.Cu at (240.0, 102.3)
- added R18: Resistor_0603_10R0, Passive:R_0603, F.Cu at (231.5, 110.7)
- added R19: Resistor_0603_10K0, Passive:R_0805, F.Cu at (227.7, 103.9)
- added R20: Resistor_0603_10K0, Passive:R_0805, F.Cu at (210.1, 119.8)
- added R21: Resistor_0603_10K0, Passive:R_0805, F.Cu at (223.3, 109.8)
- added R22: Resistor_0603_4K70, Passive:R_0603, F.Cu at (240.0, 99.8)
- added R23: Resistor_0603_4K70, Passive:R_0603, F.Cu at (227.2, 116.8)
- added R24: Resistor_0603_4K70, Passive:R_0603, F.Cu at (235.5, 108.2)
- added R25: Resistor_0603_220R, Passive:R_0603, F.Cu at (222.4, 120.5)
- added R26: Resistor_0603_220R, Passive:R_0603, F.Cu at (244.0, 99.4)
- added R27: Resistor_0603_220R, Passive:R_0603, F.Cu at (244.0, 101.9)
- added R28: Resistor_0603_470R, Passive:R_0805, F.Cu at (234.9, 97.5)
- added R29: Resistor_0603_R_DNP, Passive:R_0603, F.Cu at (231.5, 113.3)
- added R30: Resistor_0603_0R00, Passive:R_0603, F.Cu at (239.9, 104.8)
- added R31: Resistor_0603_10R0, Passive:R_0603, F.Cu at (251.6, 94.2)
- added R32: Resistor_0603_4K70, Passive:R_0603, F.Cu at (264.2, 87.6)
- added R33: Resistor_0603_4K70, Passive:R_0603, F.Cu at (235.5, 113.3)
- added R34: Resistor_0603_4K70, Passive:R_0603, F.Cu at (243.9, 106.9)
- added R35: Resistor_0603_9K10, Passive:R_0603, F.Cu at (235.2, 115.8)
- added R36: Resistor_0805_10K0, Passive:R_0805, F.Cu at (245.1, 88.9)
- added R37: Resistor_0603_1K00, Passive:R_0603, F.Cu at (252.0, 99.2)
- added R38: Resistor_0603_470R, Passive:R_0805, F.Cu at (234.9, 94.6)
- added R39: Resistor_0603_27R0, Passive:R_0603, F.Cu at (239.5, 112.4)
- added R40: Resistor_0603_27R0, Passive:R_0603, F.Cu at (231.2, 120.8)
- added R41: Resistor_0603_4K70, Passive:R_0603, F.Cu at (248.0, 104.3)
- added R42: Resistor_0603_150K, Passive:R_0603, F.Cu at (247.6, 96.8)
- added R43: Resistor_0603_10K0, Passive:R_0805, F.Cu at (223.3, 103.9)
- added R44: Resistor_0603_0R00, Passive:R_0603, F.Cu at (235.9, 105.7)
- added R6: Resistor_0805_470R, Passive:R_0805, F.Cu at (223.3, 106.9)
- added R7: Resistor_0603_39K0, Passive:R_0603, F.Cu at (243.5, 94.4)
- added R8: Resistor_0603_11K0, Passive:R_0603, F.Cu at (253.3, 88.6)
- added R9: Resistor_0805_10K0, Passive:R_0805, F.Cu at (219.0, 116.1)
- added SW1: Switch-Tact_OMRON-B3F-3100, Others:OMRON_B3F-3100, F.Cu at (101.6, 91.4)
- added SW2: Switch-Tact_OMRON-B3F-3100, Others:OMRON_B3F-3100, F.Cu at (112.4, 91.4)
- added SW3: Switch-Tact_OMRON-B3F-3100, Others:OMRON_B3F-3100, F.Cu at (90.2, 91.4)
- added TH1: NTC_0603_10K, Passive:R_0603, F.Cu at (223.2, 117.9)
- added U2: OPA_MCP6V36T-E_OT, Semiconductor:SOT-23-5, F.Cu at (218.2, 101.8)
- added U3: LDO-MCP1700T-3302E_TT-Others, Semiconductor:SOT-23, F.Cu at (214.4, 108.1)
- added U4: SENSOR_BMA250E, Semiconductor:LGA-12, F.Cu at (251.8, 102.2)
- added U5: INTERFACE_FT230XS, Semiconductor:SSOP-16, F.Cu at (152.4, 80.0)
- added U6: BATTERY_MCP73833-FCI_UN, Semiconductor:MSOP-10, F.Cu at (157.5, 95.9)
- added U7: DISPLAY_REX012832FSPP3N01, Others:RAYSTAR_REX012832, F.Cu at (98.4, 80.6)
- added Y1: Crystal_HC49SM_8MHz, Passive:Crystal_SMD_HC49-SD, F.Cu at (135.3, 70.5)
- B1: value L402036 -> BATTERY_CELLEVIA-L402036-Others; footprint Others:Battery_L402036 -> Others:CELLEVIA_L402036; moved to B.Cu
- C1, C2: value C0805_100nF -> Capacitator_0805_100nF_X7R; footprint Passive:C0805 -> Passive:C_0805
- C3: value C0805_10uF -> Capacitator_0805_10uF_X5R; footprint Passive:C0805 -> Passive:C_0805
- D1: value LED0805_KP-2012SGC -> LED_0603_Green; footprint Passive:R0805 -> Passive:LED_0603_GRE
- R1: value R0805_470R -> Resistor_0805_470R; footprint Passive:R0805 -> Passive:R_0805
- R2, R3, R4: value R0805_220R -> Resistor_0805_220R; footprint Passive:R0805 -> Passive:R_0805
- R5: value R0805_4K70 -> Resistor_0805_4K70; footprint Passive:R0805 -> Passive:R_0805
- U1: footprint Integrated Circuits:SSOP-28 -> Semiconductor:SSOP-28
- moved B1 10.9 mm to (142.2, 81.3), turned to 0 degrees
- moved C3 7.65 mm to (110.3, 73.5)
- moved R5 7.65 mm to (105.8, 76.5)
- moved C1 7.65 mm to (105.9, 73.5)
Connections:
- C1 pad 2: GND -> GNDD
- C2 pad 2: GND -> GNDD
- C3 pad 1: Net-(C3-Pad1) -> GNDD
- C3 pad 2: GND -> Net-(C3-Pad2)
- D1 pad 2: +3V3 -> +3.3VA
- J1 pad 3: GND -> GNDD
- R1 pad 2: GND -> GNDD
- U1 pad 11: Net-(U1-Pad11) -> /U1TX
- U1 pad 12: Net-(U1-Pad12) -> /U1RX
- U1 pad 14: Net-(U1-Pad14) -> /LIVE_LED
- U1 pad 15: Net-(U1-Pad15) -> /#PSEN
- U1 pad 16: /SDA -> /#RST
- U1 pad 17: /SCL -> /SCL1
- U1 pad 18: Net-(U1-Pad18) -> /SDA1
- U1 pad 19: Net-(U1-Pad19) -> GNDD
- U1 pad 2: Net-(U1-Pad2) -> /AN0
- U1 pad 20: Net-(C3-Pad1) -> Net-(C3-Pad2)
- U1 pad 21: Net-(U1-Pad21) -> /#DEN
- U1 pad 22: Net-(U1-Pad22) -> /UP
- U1 pad 23: Net-(U1-Pad23) -> /OK
- U1 pad 24: Net-(U1-Pad24) -> /DWN
- U1 pad 25: Net-(U1-Pad25) -> /#CH_CPLT
- U1 pad 27: GND -> GNDD
- U1 pad 28: +3V3 -> Net-(C15-Pad1)
- U1 pad 3: Net-(U1-Pad3) -> /AN1
- U1 pad 7: Net-(U1-Pad7) -> /INT1
- U1 pad 8: GND -> GNDD

Commit message: update
Parts:
- removed C14: Capacitator_0603_47nF_X7R, Passive:C_0603
- removed R17: Resistor_0603_9K10, Passive:R_0603
- removed R18: Resistor_0603_10R0, Passive:R_0603
- added J3: PinHeader_01x01_Male, Connectors:PinHeader_1x01_P2.54mm_Horizontal, F.Cu at (90.7, -1.52)
- added J4: PinHeader_01x01_Male, Connectors:PinHeader_1x01_P2.54mm_Horizontal, F.Cu at (5.84, -11.9)
- added J5: PinHeader_01x02_Male, Connectors:PinHeader_1x02_P2.54mm_Vertical, B.Cu at (85.9, -22.1)
- added L3: Filter_0603_CB03YTYH101, Passive:L_0603, F.Cu at (82.8, -13.2)
- added R45: Resistor_0603_1K00, Passive:R_0603, F.Cu at (71.6, -11.4)
- B1: value BATTERY_CELLEVIA-L402036-Others -> BATTERY_L402036
- C1, C10, C11, C2, C6, C8: value Capacitator_0805_100nF_X7R -> Capacitator_0603_100nF_X7R; footprint Passive:C_0805 -> Passive:C_0603
- C12, C16, C26, C34, C35, C36, C9: value Capacitator_0805_1uF_X7R -> Capacitator_0603_1uF_X7R
- C3: value Capacitator_0805_10uF_X5R -> Capacitator_0603_10uF_X5R; footprint Passive:C_0805 -> Passive:C_0603
- C4, C5: value Capacitator_0805_22pF_X7R -> Capacitator_0603_22pF_NP0; footprint Passive:C_0805 -> Passive:C_0603
- J1: value PinStrip_01x06_Male -> PinHeader_01x06_Male; footprint Connectors:PinStrip_1x06_P2.54mm_Vertical -> Connectors:PinHeader_1x06_P2.54mm_Vertical
- R1, R12, R6: value Resistor_0805_470R -> Resistor_0603_470R; footprint Passive:R_0805 -> Passive:R_0603
- R10, R14, R36, R9: value Resistor_0805_10K0 -> Resistor_0603_10K0; footprint Passive:R_0805 -> Passive:R_0603
- R11: value Resistor_0805_R_DNP -> Resistor_0603_R_DNP; footprint Passive:R_0805 -> Passive:R_0603
- R13: value Resistor_0805_0R00 -> Resistor_0603_0R00; footprint Passive:R_0805 -> Passive:R_0603
- R16: value Resistor_0603_4K70 -> Resistor_0603_0R00
- R19, R20, R21, R28, R38, R43: footprint Passive:R_0805 -> Passive:R_0603
- R2, R3, R4: value Resistor_0805_220R -> Resistor_0603_220R; footprint Passive:R_0805 -> Passive:R_0603
- R44: value Resistor_0603_0R00 -> Resistor_0603_220R
- R5: value Resistor_0805_4K70 -> Resistor_0603_4K70; footprint Passive:R_0805 -> Passive:R_0603
- U3: value LDO-MCP1700T-3302E_TT-Others -> LDO_MCP1700T-3302E_TT
- Y1: value Crystal_HC49SM_8MHz -> Crystal_SMD3225_12MHz; footprint Passive:Crystal_SMD_HC49-SD -> Passive:Crystal_SMD_3225
- moved R8 269.6 mm to (1.78, -8.38), turned to 180 degrees
- moved R11 267.7 mm to (1.78, -15.5)
- moved R7 259.0 mm to (5.84, -8.38)
- moved R16 258.8 mm to (9.65, -7.62)
- moved R10 258.8 mm to (5.84, -17.0), turned to 180 degrees
- moved C7 257.3 mm to (1.78, -19.6), turned to 180 degrees
- moved R12 256.3 mm to (5.84, -20.6), turned to 180 degrees
- moved C10 254.0 mm to (9.65, -9.14), turned to 180 degrees
- moved C6 251.8 mm to (1.78, -17.5), turned to 180 degrees
- moved R32 251.4 mm to (32.8, -10.7), turned to 270 degrees
- moved R9 248.9 mm to (11.7, -21.6), turned to 270 degrees
- moved C11 247.6 mm to (10.7, -18.8), turned to 180 degrees
- moved C22 246.5 mm to (29.7, -10.7), turned to 270 degrees
- moved Q2 245.9 mm to (10.2, -13.7)
- moved C17 244.8 mm to (20.6, -10.7), turned to 90 degrees
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Connections:
- net /#CH_CPLT renamed /CH_CPLT#
- net /#DEN renamed /DEN#
- net /#MCLR renamed /MCLR#
- net /#PSEN renamed /PSEN#
- net /DWN renamed /DN#
- net /OK renamed /OK#
- net /UP renamed /UP#
- F1 pad 2: Net-(B1-Pad1) -> Net-(F1-Pad2)
- J2 pad 1: /5V_USB -> Net-(J2-Pad1)
- Q3 pad 1: /#PG -> Net-(Q3-Pad1)
- R14 pad 2: /#PG -> Net-(Q3-Pad1)
- R16 pad 1: +BATT -> Net-(R15-Pad1)
- R44 pad 1: GNDD -> /RST#
- R44 pad 2: Net-(B1-Pad2) -> Net-(R44-Pad2)
- U1 pad 16: /#RST -> /RST#
- U2 pad 4: Net-(R15-Pad1) -> Net-(R16-Pad2)
- U6 pad 7: /#PG -> /PG#
- U7 pad 5: +BATT -> +3V3
- U7 pad 9: /#RST -> Net-(R44-Pad2)
- Y1 pad 2: Net-(C5-Pad1) -> GNDD
Routing:
- net +3V3: track 0.00 -> 207.7 mm, vias 0 -> 13
- net GNDD: track 0.00 -> 158.5 mm, vias 0 -> 22
- net +BATT: track 0.00 -> 66.3 mm, vias 0 -> 3
- net /PSEN#: track 0.00 -> 58.6 mm, vias 0 -> 2
- net /IC1: track 0.00 -> 56.8 mm, vias 0 -> 4
- net /SDA1: track 0.00 -> 54.4 mm, vias 0 -> 3
- net /SCL1: track 0.00 -> 50.6 mm, vias 0 -> 3
- net /DN#: track 0.00 -> 46.9 mm, vias 0 -> 2
- net Net-(R15-Pad1): track 0.00 -> 44.6 mm, vias 0 -> 2
- net /OK#: track 0.00 -> 41.0 mm, vias 0 -> 2
- net +3.3VA: track 0.00 -> 39.0 mm, vias 0 -> 2
- net /UP#: track 0.00 -> 37.2 mm, vias 0 -> 2
- net /MCLR#: track 0.00 -> 30.2 mm, vias 0 -> 2
- net Net-(J1-Pad6): track 27.3 -> 0.00 mm, vias 3 -> 0
- net /CH_CPLT#: track 0.00 -> 24.2 mm, vias 0 -> 2
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- added copper zone on B.Cu, net GNDD
Other:
- board size 88.9 x 23.5 mm -> 95 x 24 mm
- net class Default: clearance 0.2 -> 0.1778; trace_width 0.25 -> 0.254; via_dia 0.8 -> 0.635; via_drill 0.4 -> 0.4064
- rule trace_clearance: 0.2 -> 0.1778

Commit message: update
Parts:
- moved B1 166.4 mm to (163.8, 82.0)
- moved C15 139.1 mm to (155.4, 74.9)
- moved C16 139.1 mm to (153.9, 74.9)
- moved C27 139.1 mm to (180.8, 85.6)
- moved C34 139.1 mm to (178.6, 81.5)
- moved D6 139.1 mm to (172.5, 72.6)
- moved F1 139.1 mm to (178.6, 73.4)
- moved J3 139.1 mm to (191.8, 94.0)
- moved R36 139.1 mm to (149.1, 83.6)
- moved R37 139.1 mm to (178.6, 83.0)
- moved R41 139.1 mm to (157.0, 74.9)
- moved R43 139.1 mm to (172.5, 74.2)
- moved SW3 139.1 mm to (129.0, 92.7)
- moved U5 139.1 mm to (180.1, 90.2)
- moved Y1 139.1 mm to (165.4, 89.9)
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Routing:
- net +3.3VA: track 39.0 -> 40.5 mm
- added copper zone on B.Cu, net Net-(C8-Pad2)
Other:
- board text added: "MLGC210815V00"
- board text added: "SMART LOGIC PROBE"

Commit message: update
Parts:
- U7: value DISPLAY_REX012832FSPP3N01 -> DISPLAY_REX012832FWPP3N01
Connections:
- U4 pad 4: Net-(U4-Pad4) -> GNDD
- U7 pad 5: +3V3 -> Net-(C29-Pad1)
- U7 pad 6: Net-(C29-Pad1) -> Net-(U7-Pad6)
Routing:
- net +3V3: track 207.7 -> 193.6 mm
- net /UP#: track 37.2 -> 41.4 mm
- net GNDD: track 158.5 -> 157.5 mm
- net /SDA1: track 54.4 -> 53.6 mm
